File: hardware/blueboard/blueboard.kicad_pcb (KiCad board)
At the start: 2 copper layers, 199.4 x 198.9 mm, 107 parts, among them SW1 SW_SPST

Commit message: too many changes to remember
Parts:
- removed the WireConnection_1-2mmDrill at (83.2, 85.7)
- removed the WireConnection_1-2mmDrill at (311.7, 71.0)
- moved LED12 165.9 mm to (215.5, 100.3)
- moved R12 151.4 mm to (214.6, 87.8)
- moved LED13 150.0 mm to (164.1, 108.7)
- moved LED5 146.7 mm to (214.8, -75.9)
- moved LED10 137.9 mm to (272.0, 101.6)
- moved R5 131.9 mm to (213.9, -60.5), turned to 90 degrees
- moved R13 129.7 mm to (163.1, 88.7)
- moved R11 121.0 mm to (110.4, 86.2)
- moved LED11 119.9 mm to (111.3, 101.1)
- moved LED16 119.1 mm to (216.0, 41.8)
- moved R10 117.2 mm to (271.0, 87.1), turned to 270 degrees
- moved R16 115.5 mm to (215.1, 60.7), turned to 90 degrees
- moved LED8 107.7 mm to (271.5, 43.1)
- moved R15 103.3 mm to (162.6, 63.2), turned to 90 degrees
- moved LED15 102.3 mm to (163.5, 50.3)
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Routing:
- net GND: track 33.3 -> 923.0 mm, vias 0 -> 2
- net G: track 16.2 -> 872.0 mm, vias 1 -> 0
- net R: track 16.5 -> 869.1 mm, vias 1 -> 0
- net B: track 64.0 -> 867.7 mm, vias 1 -> 0
- net 5V: track 715.6 -> 908.8 mm
- net Net-(R4-Pad1): track 0.00 -> 166.4 mm, vias 0 -> 1
- net Net-(R10-Pad1): track 0.00 -> 165.8 mm, vias 0 -> 1
- net Net-(R6-Pad1): track 0.00 -> 141.7 mm
- net Net-(R8-Pad1): track 0.00 -> 139.8 mm, vias 0 -> 1
- net Net-(R12-Pad1): track 0.00 -> 123.6 mm, vias 0 -> 1
- net Net-(JP2-Pad6): track 9.70 -> 132.9 mm, vias 0 -> 1
- net Net-(R5-Pad1): track 0.00 -> 113.9 mm, vias 0 -> 1
- net Net-(R11-Pad1): track 0.00 -> 110.2 mm
- net Net-(R97-Pad2): track 0.00 -> 108.5 mm, vias 0 -> 1
- net Net-(R16-Pad1): track 0.00 -> 106.4 mm, vias 0 -> 1
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- removed copper zone on B.Cu, net GND
- removed copper zone on F.Cu, net GND

Commit message: round 2 of board design
Parts:
- removed LOGO_OSHW_silkscreen_10mm: val**, Freetronics:LOGO_OSHW_silkscreen_10mm
- removed WireConnection_1-2mmDrill: VAL**, Wire_Connections_Bridges:WireConnection_1-2mmDrill
- added JP10: M01, Freetronics:1X01, F.Cu at (210.6, 19.3)
- added JP11: M01, Freetronics:1X01, F.Cu at (191.4, 19.1)
- added JP12: M01, Freetronics:1X01, F.Cu at (188.6, 19.1)
- added JP13: M01, Freetronics:1X01, F.Cu at (186.0, 19.2)
- added JP14: M01, Freetronics:1X01, F.Cu at (183.5, 19.2)
- added JP15: M01, Freetronics:1X01, F.Cu at (180.9, 19.1)
- added JP16: M01, Freetronics:1X01, F.Cu at (171.3, 19.5)
- added JP17: M01, Freetronics:1X01, F.Cu at (168.6, 19.4)
- added JP18: M01, Freetronics:1X01, F.Cu at (165.9, 19.5)
- added JP19: M01, Freetronics:1X01, F.Cu at (163.2, 19.5)
- added JP20: M01, Freetronics:1X01, F.Cu at (145.6, 19.2)
- added JP21: M01, Freetronics:1X01, F.Cu at (143.0, 19.1)
- added JP22: M01, Freetronics:1X01, F.Cu at (183.0, 120.8)
- added JP3: M01, Freetronics:1X01, F.Cu at (140.1, -26.1)
- added JP4: M01, Freetronics:1X01, F.Cu at (148.9, -26.2)
- added JP5: M01, Freetronics:1X01, F.Cu at (140.2, -23.2)
- added JP6: M01, Freetronics:1X01, F.Cu at (148.9, -23.3)
- added Q1: TRANSISTOR_NPN, finn_kicad:EBC-transistor-NPN, F.Cu at (200.4, 25.6)
- added Q2: TRANSISTOR_NPN, finn_kicad:EBC-transistor-NPN, F.Cu at (186.3, 25.7)
- added Q3: TRANSISTOR_NPN, finn_kicad:EBC-transistor-NPN, F.Cu at (215.0, 25.6)
- added R17: 10k, Resistors_ThroughHole:Resistor_Horizontal_RM10mm, F.Cu at (199.7, -72.1)
- added SW2: SW_PUSHBUTTON, Freetronics:1X02, F.Cu at (199.7, -81.0)
- JP2: value M07 -> M01
- R98: value R -> 2.2k
- SW1: footprint Freetronics:SW_PUSHBUTTON_TC0122 -> Freetronics:1X02
- moved R59 14.1 mm to (243.5, -14.0)
- moved JP2 0.39 mm to (293.0, -36.4)
Connections:
- JP2 pad 1: Net-(JP1-Pad1) -> Net-(JP2-Pad1)
- JP2 pad 2: Net-(JP2-Pad2) -> (no net)
- JP2 pad 3: 5V -> (no net)
- JP2 pad 4: GND -> (no net)
- JP2 pad 5: Net-(JP2-Pad5) -> (no net)
- JP2 pad 6: Net-(JP2-Pad6) -> (no net)
- JP2 pad 7: Net-(JP2-Pad7) -> (no net)
- R1 pad 2: Net-(LED1-PadA) -> Net-(LED16-PadA)
- R10 pad 2: Net-(LED10-PadA) -> Net-(LED9-PadA)
- R11 pad 2: Net-(LED11-PadA) -> Net-(LED10-PadA)
- R12 pad 2: Net-(LED12-PadA) -> Net-(LED11-PadA)
- R13 pad 1: Net-(R13-Pad1) -> Net-(LED15-PadA)
- R13 pad 2: Net-(LED13-PadA) -> Net-(R13-Pad2)
- R14 pad 1: Net-(R14-Pad1) -> Net-(LED14-PadA)
- R14 pad 2: Net-(LED14-PadA) -> Net-(R14-Pad2)
- R15 pad 1: Net-(R15-Pad1) -> Net-(LED13-PadA)
- R15 pad 2: Net-(LED15-PadA) -> Net-(R15-Pad2)
- R16 pad 1: Net-(R16-Pad1) -> Net-(LED12-PadA)
- R16 pad 2: Net-(LED16-PadA) -> Net-(R16-Pad2)
- R2 pad 2: Net-(LED2-PadA) -> Net-(LED1-PadA)
- R3 pad 2: Net-(LED3-PadA) -> Net-(LED2-PadA)
- R4 pad 2: Net-(LED4-PadA) -> Net-(LED3-PadA)
- R5 pad 2: Net-(LED5-PadA) -> Net-(LED4-PadA)
- R6 pad 2: Net-(LED6-PadA) -> Net-(LED5-PadA)
- R7 pad 2: Net-(LED7-PadA) -> Net-(LED6-PadA)
- R8 pad 2: Net-(LED8-PadA) -> Net-(LED7-PadA)
- R9 pad 2: Net-(LED9-PadA) -> Net-(LED8-PadA)
- R97 pad 1: Net-(JP2-Pad5) -> Net-(R97-Pad1)
- R98 pad 1: Net-(JP2-Pad5) -> GND
- R98 pad 2: GND -> Net-(R97-Pad1)
- SHIELD1 pad 10: Net-(JP2-Pad6) -> Net-(SHIELD1-Pad10)
- SHIELD1 pad 34: Net-(R16-Pad1) -> Net-(R13-Pad2)
- SHIELD1 pad 35: Net-(R15-Pad1) -> Net-(R14-Pad2)
- SHIELD1 pad 36: Net-(R14-Pad1) -> Net-(R15-Pad2)
- SHIELD1 pad 37: Net-(R13-Pad1) -> Net-(R16-Pad2)
- SHIELD1 pad 3V3: Net-(SHIELD1-Pad3V3) -> Net-(JP2-Pad1)
- SHIELD1 pad RST: Net-(SHIELD1-PadRST) -> Net-(JP1-Pad1)
Routing:
- net GND: track 923.0 -> 0.00 mm, vias 2 -> 0
- net 5V: track 908.8 -> 0.00 mm
- net G: track 872.0 -> 0.00 mm
- net R: track 869.1 -> 0.00 mm
- net B: track 867.7 -> 0.00 mm
- net Net-(R67-Pad2): track 197.3 -> 0.00 mm
- net Net-(R53-Pad1): track 192.8 -> 0.00 mm
- net Net-(R61-Pad1): track 174.2 -> 0.00 mm
- net Net-(R77-Pad2): track 172.7 -> 0.00 mm, vias 1 -> 0
- net Net-(R81-Pad2): track 169.0 -> 0.00 mm
- net Net-(R4-Pad1): track 166.4 -> 0.00 mm, vias 1 -> 0
- net Net-(R10-Pad1): track 165.8 -> 0.00 mm, vias 1 -> 0
- net Net-(R95-Pad2): track 164.2 -> 0.00 mm, vias 1 -> 0
- net Net-(R85-Pad2): track 155.6 -> 0.00 mm, vias 1 -> 0
- net Net-(R55-Pad1): track 153.3 -> 0.00 mm
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