File: hardware/blueboard/blueboard_orig.sch (KiCad schematic (older format))
At the start: 126 parts, among them Q1 TRANSISTOR_NPN, Q2 TRANSISTOR_NPN, Q3 TRANSISTOR_NPN, SW1 SW_SPST, SW2 SW_PUSHBUTTON

Commit message: round 2 of board design
Parts:
- removed HC1: HC05, MODULE, symbol HC05
- removed JP10, JP11, JP12, JP13, JP14, JP15, JP16, JP17, JP18, JP19, JP20, JP21, JP22, JP3, JP4, JP5, JP6: M01, Freetronics:1X01, symbol M01
- removed JP2: M01, Freetronics:1X07, symbol M01
- removed Q1, Q2, Q3: TRANSISTOR_NPN, finn_kicad:EBC-transistor-NPN, symbol TRANSISTOR_NPN
- removed R17: 10k, Resistors_ThroughHole:Resistor_Horizontal_RM10mm, symbol R
- removed SW2: SW_PUSHBUTTON, Freetronics:1X02, symbol SW_PUSHBUTTON
- added JP2: M07, Freetronics:1X07, symbol M07
- R98: value 2.2k -> R
- SW1: footprint Freetronics:1X02 -> Freetronics:SW_PUSHBUTTON_TC0122
Connections:
- net 5V: now also JP2.3
- net GND: now also R98.2, JP2.4; no longer R98.1
- net at SHIELD1.10: now also JP2.6
- net at SHIELD1.34 (PC3): now also R16.1; no longer R13.2
- net at SHIELD1.35 (PC2): now also R15.1; no longer R14.2
- net at SHIELD1.36 (PC1): now also R14.1; no longer R15.2
- net at SHIELD1.37 (PC0): now also R13.1; no longer R16.2
- net at SHIELD1.RST: no longer JP1.1
- net at LED13.A: now also R13.2; no longer R15.1
- net at LED12.A: now also R12.2; no longer R16.1
- net at LED15.A: now also R15.2; no longer R13.1
- net at LED14.A: now also R14.2; no longer R14.1
- net at R1.2: now also LED1.A; no longer LED16.A
- net at LED9.A: now also R9.2; no longer R10.2
- net at LED11.A: now also R11.2; no longer R12.2
- net at LED10.A: now also R10.2; no longer R11.2
- net at LED6.A: now also R6.2; no longer R7.2
- net at LED5.A: now also R5.2; no longer R6.2
- net at LED8.A: now also R8.2; no longer R9.2
- net at LED7.A: now also R7.2; no longer R8.2
- net at LED2.A: now also R2.2; no longer R3.2
- net at LED4.A: now also R4.2; no longer R5.2
- net at LED3.A: now also R3.2; no longer R4.2
- net at R97.1: now also R98.1, JP2.5; no longer R98.2
- new net: JP1.1, JP2.1
- new net: LED16.A, R16.2
- no-connect marks 9 -> 0
Other:
- moved on the sheet: R97, R98
